File: megamesh_node_v1_0/megamesh_node_v1_0.kicad_sch (KiCad schematic)
At the start: 53 parts, among them J1 Conn_Coaxial, J2 Screw_Terminal_01x02, J3 Screw_Terminal_01x02, P1 USB_C_Plug_USB2.0, Q1 CSD87312Q3E, Q2 CSD87312Q3E, U1 ESP32-S3-WROOM-1, U2 LoRa126XF30, U3 BQ25798, U4 TPS63001

Commit message: Entwicklung Schaltplan und Platine
Es geht voran
Parts:
- removed C18, C19: 33 uF POSCAP, symbol Device:C
- removed U4: TPS63001, Package_SON:Texas_DRC0010J_ThermalVias, symbol Regulator_Switching:TPS63001
- added C26, C33: 100 nF, Capacitor_SMD:C_0603_1608Metric, symbol Device:C
- added C27, C28: 1 uF, Capacitor_SMD:C_0603_1608Metric, symbol Device:C
- added C29, C30, C31, C32: 22 uF, Capacitor_SMD:C_0805_2012Metric, symbol Device:C
- added C34: 10 uF, Capacitor_SMD:C_0805_2012Metric, symbol Device:C
- added GND1, GND2, GND3: GND, TestPoint:TestPoint_THTPad_2.0x2.0mm_Drill1.0mm, symbol Connector:TestPoint
- added GP1: GPIO1, TestPoint:TestPoint_THTPad_D2.0mm_Drill1.0mm, symbol Connector:TestPoint
- added GP15: I2C SDA, TestPoint:TestPoint_THTPad_D2.0mm_Drill1.0mm, symbol Connector:TestPoint
- added GP16: I2C SCL, TestPoint:TestPoint_THTPad_D2.0mm_Drill1.0mm, symbol Connector:TestPoint
- added GP17: GPIO17, TestPoint:TestPoint_THTPad_D2.0mm_Drill1.0mm, symbol Connector:TestPoint
- added GP18: GPIO18, TestPoint:TestPoint_THTPad_D2.0mm_Drill1.0mm, symbol Connector:TestPoint
- added GP2: GPIO2, TestPoint:TestPoint_THTPad_D2.0mm_Drill1.0mm, symbol Connector:TestPoint
- added GP21: GPIO21, TestPoint:TestPoint_THTPad_D2.0mm_Drill1.0mm, symbol Connector:TestPoint
- added GP3: GPIO3, TestPoint:TestPoint_THTPad_D2.0mm_Drill1.0mm, symbol Connector:TestPoint
- added GP38: GPIO38, TestPoint:TestPoint_THTPad_D2.0mm_Drill1.0mm, symbol Connector:TestPoint
- added GP39: GPIO39, TestPoint:TestPoint_THTPad_D2.0mm_Drill1.0mm, symbol Connector:TestPoint
- added GP4: GPIO4, TestPoint:TestPoint_THTPad_D2.0mm_Drill1.0mm, symbol Connector:TestPoint
- added GP40: GPIO40, TestPoint:TestPoint_THTPad_D2.0mm_Drill1.0mm, symbol Connector:TestPoint
- added GP41: GPIO41, TestPoint:TestPoint_THTPad_D2.0mm_Drill1.0mm, symbol Connector:TestPoint
- added GP42: GPIO42, TestPoint:TestPoint_THTPad_D2.0mm_Drill1.0mm, symbol Connector:TestPoint
- added GP43: TX0, TestPoint:TestPoint_THTPad_D2.0mm_Drill1.0mm, symbol Connector:TestPoint
- added GP44: RX0, TestPoint:TestPoint_THTPad_D2.0mm_Drill1.0mm, symbol Connector:TestPoint
- added GP47: GPIO47, TestPoint:TestPoint_THTPad_D2.0mm_Drill1.0mm, symbol Connector:TestPoint
- added GP48: GPIO48, TestPoint:TestPoint_THTPad_D2.0mm_Drill1.0mm, symbol Connector:TestPoint
- added L2, L3: 1.5 uH, myRF:IND-SMD_L4.2-W4.0_SPM4030T, symbol Device:L
- added R15: 200 kOhm, Capacitor_SMD:C_0603_1608Metric, symbol Device:R
- added R16: 624 kOhm, Capacitor_SMD:C_0603_1608Metric, symbol Device:R
- added R17, R19: 10 kOhm, Capacitor_SMD:C_0603_1608Metric, symbol Device:R
- added R20: 649 kOhm, Capacitor_SMD:C_0603_1608Metric, symbol Device:R
- added R21: 100 kOhm, Capacitor_SMD:C_0603_1608Metric, symbol Device:R
- added SW1, SW3: SW_Push, myRF:SW_TS-1088-AR02016, symbol Switch:SW_Push
- added U4, U5: TPS63070RNMR, TPS63070RNMR:VREG_TPS63070RNMR, symbol myRF:TPS63070RNMR
- added VCC1, VCC2, VCC3: 3v3, TestPoint:TestPoint_THTPad_D2.0mm_Drill1.0mm, symbol Connector:TestPoint
- C1: value 47uF -> 47 uF; footprint (none) -> Capacitor_SMD:C_1206_3216Metric; symbol Device:C_Polarized -> Device:C
- C10, C9: footprint (none) -> Capacitor_SMD:C_1206_3216Metric
- C11, C14, C25, C3, C4, C5, C6, R1, R10, R11, R12, R13, R14, R2, R4, R5, R6, R7, R8, R9: footprint (none) -> Capacitor_SMD:C_0603_1608Metric
- C12, C13, C15, C16, C17, C20, C21, C22, C23, C24, C7, C8: footprint (none) -> Capacitor_SMD:C_0805_2012Metric
- C2: value 100nF -> 100 nF; footprint (none) -> Capacitor_SMD:C_0603_1608Metric
- D3: footprint (none) -> myRF:LED-SMD_L1.7-W0.6-R-RD
- J2, J3: footprint (none) -> myRF:CONN-TH_2P-P3.81_KF124-3.81-2P
- L1: footprint (none) -> myRF:IND-SMD_L7.1-W6.5-P5.60
- P1: footprint (none) -> Connector_USB:USB_C_Receptacle_HRO_TYPE-C-31-M-12
- Q1, Q2: footprint (none) -> myRF:SON 3.3x3.3mm
- R3: value R -> 5.1 kOhm; footprint (none) -> Capacitor_SMD:C_0603_1608Metric
Connections:
- net +3V3: now also C29.1, C30.1, C33.1, C34.1, R16.1, R17.1, R19.1, U5.7_8 (VOUT), VCC1.1, VCC2.1, VCC3.1
- net GND: now also U2.8 (GND), C26.2, C27.2, C28.2, C29.2, C30.2, C31.2, C32.2, C33.2, C34.2, GND1.1, GND2.1, GND3.1, R15.2, R21.2, SW1.1, SW3.2, U4.10 (PGND), U4.15 (VSEL), U4.4 (GND), U4.6 (FB2), U5.10 (PGND), U5.15 (VSEL), U5.4 (GND), U5.6 (FB2)
- net SYS: now also U4.1 (PS/SYNC), U4.12_13 (VIN), U4.14 (EN), U5.1 (PS/SYNC), U5.12_13 (VIN), U5.14 (EN)
- net Gate_ACDRV2: now reaches R2.1, U3.10 (ACDRV2)
- net Gate_ACDRV1: now reaches R1.1, U3.11 (ACDRV1)
- net D2: now reaches C4.1, C7.1, C8.1, Q1.6 (D2), Q1.7 (D2), Q1.8 (D2), Q2.6 (D2), Q2.7 (D2), Q2.8 (D2), U3.2 (VBUS), U3.3 (VBUS)
- net !INT: now reaches R14.2, U1.5 (GPIO5/TOUCH5/ADC1_CH4), U3.21 (~{INT})
- net REGN: now reaches C11.2, R7.2, U3.5 (REGN)
- net REGN: now also R12.1, R8.1
- net D1_VAC2: now reaches C5.1, J2.1 (Pin_1), Q2.1 (D1), Q2.2 (D1), Q2.3 (D1), Q2.4 (D1), U3.8 (VAC2)
- net D1_VAC1: now reaches C3.1, P1.A4 (VBUS), P1.A9 (VBUS), P1.B4 (VBUS), P1.B9 (VBUS), Q1.1 (D1), Q1.2 (D1), Q1.3 (D1), Q1.4 (D1), R4.1, U3.9 (VAC1)
- net D+: now reaches P1.A6 (D+), U1.14 (GPIO20/U1CTS/ADC2_CH9/CLK_OUT1/USB_D+)
- net D-: now reaches P1.A7 (D-), U1.13 (GPIO19/U1RTS/ADC2_CH8/CLK_OUT2/USB_D-)
- net at U1.10 (GPIO17/U1TXD/ADC2_CH6): now also GP17.1
- net at U1.11 (GPIO18/U1RXD/ADC2_CH7/CLK_OUT3): now also GP18.1
- net at U1.15 (GPIO3/TOUCH3/ADC1_CH2): now also GP3.1
- net MOSI: now reaches U1.18 (GPIO10/TOUCH10/ADC1_CH9/FSPICS0/FSPIIO4/SUBSPICS0)
- net MOSI: now also U2.11 (MOSI)
- net MISO: now reaches U1.19 (GPIO11/TOUCH11/ADC2_CH0/FSPID/FSPIIO5/SUBSPID)
- net MISO: now also U2.10 (MISO)
- net NRESET: now reaches U1.20 (GPIO12/TOUCH12/ADC2_CH1/FSPICLK/FSPIIO6/SUBSPICLK)
- net NRESET: now also U2.5 (NRESET)
- net BUSY: now reaches U1.21 (GPIO13/TOUCH13/ADC2_CH2/FSPIQ/FSPIIO7/SUBSPIQ)
- net BUSY: now also U2.6 (BUSY)
- net DIO0: now reaches U1.22 (GPIO14/TOUCH14/ADC2_CH3/FSPIWP/FSPIDQS/SUBSPIWP)
- net DIO0: now also U2.13 (DIO1)
- net at U1.23 (GPIO21): now also GP21.1
- net at U1.24 (GPIO47/SPICLK_P/SUBSPICLK_P_DIFF): now also GP47.1
- net at U1.25 (GPIO48/SPICLK_N/SUBSPICLK_N_DIFF): now also GP48.1
- net BOOT_SW: now reaches U1.27 (GPIO0/BOOT)
- net BOOT_SW: now also R19.2, SW3.1
- net EN_SW: now reaches U1.3 (EN)
- net EN_SW: now also C26.1, R17.2, SW1.2
- net at U1.31 (GPIO38/FSPIWP/SUBSPIWP): now also GP38.1
- net at U1.32 (MTCK/GPIO39/CLK_OUT3/SUBSPICS1): now also GP39.1
- net at U1.33 (MTDO/GPIO40/CLK_OUT2): now also GP40.1
- net at U1.34 (MTDI/GPIO41/CLK_OUT1): now also GP41.1
- net at U1.35 (MTMS/GPIO42): now also GP42.1
- net at U1.36 (U0RXD/GPIO44/CLK_OUT2): now also GP44.1
- net at U1.37 (U0TXD/GPIO43/CLK_OUT1): now also GP43.1
- net at U1.38 (GPIO2/TOUCH2/ADC1_CH1): now also GP2.1
- net at U1.39 (GPIO1/TOUCH1/ADC1_CH0): now also GP1.1
- net at U1.4 (GPIO4/TOUCH4/ADC1_CH3): now also GP4.1; no longer U2.13 (DIO1)
- net SDA: now reaches U1.6 (GPIO6/TOUCH6/ADC1_CH5)
- net SDA: now also R6.2, U3.15 (SDA)
- net SCL: now reaches U1.7 (GPIO7/TOUCH7/ADC1_CH6)
- net SCL: now also R5.2, U3.14 (SCL)
- net at U1.8 (GPIO15/U0RTS/ADC2_CH4/XTAL_32K_P): now also GP15.1
- net at U1.9 (GPIO16/U0CTS/ADC2_CH5/XTAL_32K_N): now also GP16.1
- net NSS: now reaches U2.7 (NSS)
- net NSS: now also U1.12 (GPIO8/TOUCH8/ADC1_CH7/SUBSPICS1)
- net SCK: now reaches U2.9 (SCK)
- net SCK: now also U1.17 (GPIO9/TOUCH9/ADC1_CH8/FSPIHD/SUBSPIHD)
- net +5V renamed +6V
- net +6V: now also C31.1, C32.1, R20.1, U4.7_8 (VOUT)
- new net: L3.1, U4.9 (L2)
- new net: L3.2, U4.11 (L1)
- new net: C28.1, U4.3 (VAUX)
- new net: L2.2, U5.11 (L1)
- new net: C27.1, U5.3 (VAUX)
- new net: R15.1, R16.2, U5.5 (FB)
- new net: L2.1, U5.9 (L2)
- new net: R20.2, R21.1, U4.5 (FB)
Other:
- note added: "3.3 Volt Buck-Boost Converter"
- note added: "6 Volt Buck-Boost Converter"
- note added: "Back to Back NFETs"
- note added: "Boot Switch"
- note added: "Buck-Boost Converters"
- note added: "Buck-Boost Solar Charging Controller"
- note added: "ESP32-S3-WROOM-1"
- note added: "LoRa Module"
- note added: "Power Decoupling"
- note added: "Reset Switch"
- note added: "Solar Power"
- note added: "Switches"
- note added: "To Battery"
- note added: "USB Port and Power Selection"
- note added: "USB Power"
- note removed: "Back to Back Mosfetz"
- note removed: "Für PV"
- note removed: "Für USB"
- moved on the sheet: C10, C11, C12, C13, C14, C15, C16, C17, C2, C20, C21, C22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
